File: KiCad/Battery-Tester.kicad_pcb (KiCad board)
At the start: 2 copper layers, 31 parts, among them J1 Conn_01x02, J3 Conn_01x07, Q1 SI2304, Q2 SI2304, Q3 SI2304, Q4 SI2304, U1 MCP6001-OT

Commit message: Minor modifications.
Parts:
- added Q5: Si2347DS, Package_TO_SOT_SMD:SOT-23, F.Cu at (96.0, 127.0)
- added Q6: Si2347DS, Package_TO_SOT_SMD:SOT-23, F.Cu at (110.0, 89.5)
- Q1, Q2, Q3, Q4: value SI2304 -> SI2304DDS
- moved R17 27.0 mm to (84.8, 89.5), turned to 90 degrees
- moved D2 22.5 mm to (87.0, 89.5), turned to 90 degrees
- moved JP1 4.00 mm to (101.0, 126.5)
- moved R3 4.00 mm to (108.9, 126.5)
- moved J3 1.50 mm to (106.0, 89.5)
Connections:
- J3 pad 1: +5V -> Net-(J3-Pad1)
- JP1 pad 1: Net-(J1-Pad1) -> Net-(JP1-Pad1)
- R1 pad 2: Net-(J1-Pad1) -> Net-(JP1-Pad1)
Routing:
- net Net-(JP1-Pad1): track 0.00 -> 9.80 mm
- net Net-(J1-Pad1): track 12.1 -> 4.21 mm
- net Net-(J3-Pad1): track 0.00 -> 3.39 mm
- net +5V: track 65.6 -> 68.0 mm
- net GND: track 18.5 -> 20.6 mm, vias 10 -> 12
- net Net-(F1-Pad1): track 7.02 -> 5.15 mm
- net Net-(J3-Pad5): track 12.4 -> 13.9 mm
- net Net-(J3-Pad4): track 8.55 -> 10.0 mm
- net Net-(J3-Pad3): track 6.47 -> 7.97 mm
- net Net-(J3-Pad2): track 10.4 -> 11.9 mm
- net Net-(C3-Pad1): track 34.1 -> 35.6 mm
Other:
- board outline added: 32 x 44 mm
- rule solder_mask_min_width: 0.25 -> 0.15
- board text added: "+5V"
- board text added: "-BAT+"
- board text added: "GND"
- board text added: "Isns"
- board text added: "Q1"
- board text added: "Q2"
- board text added: "Q3"
- board text added: "Q4"
- board text added: "Vsns"
